File: main_low_pass.sch (EAGLE design)
At the start: 8 parts, among them IC1 74HC14D, U1 LM358PW

Commit message: Board update, alles moet nog nagemeten ed worden.
Parts:
- added JP3: (no value), pinhead:PINHD-1X3
- JP1, JP2: device pinhead:PINHD-1X3 -> pinhead:PINHD-1X4
- R1: value 6.8k -> (none)
Connections:
- new net N$5: JP3.2, SV1.3
- net GND: now also JP1.2, JP1.3, JP2.4, JP3.1
- net N$1: now also JP2.2, JP2.3; no longer SV1.3
- net N$6: now also JP1.4, JP2.1, JP3.3
Changed lines of the file:
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@@
 <part name="GND1" library="supply1" deviceset="GND" device=""/>
 <part name="SV1" library="con-lstb" deviceset="MA05-1" device=""/>
-<part name="R1" library="resistor" deviceset="R-EU_" device="R1005" value="6.8k"/>
+<part name="R1" library="resistor" deviceset="R-EU_" device="R1005"/>
 <part name="R2" library="resistor" deviceset="R-EU_" device="R1005" value="15k"/>
 <part name="GND2" library="supply1" deviceset="GND" device=""/>
 <part name="C1" library="resistor" deviceset="CPOL-EU" device="085CS-1AR" value="15u"/>
-<part name="U1" library="untitled" deviceset="LM358PW" device=""/>
+<part name="U1" library="untitled" deviceset="LM358PW" device="" value=""/>
 <part name="GND3" library="supply1" deviceset="GND" device=""/>
-<part name="JP1" library="pinhead" deviceset="PINHD-1X3" device=""/>
-<part name="JP2" library="pinhead" deviceset="PINHD-1X3" device=""/>
+<part name="JP1" library="pinhead" deviceset="PINHD-1X4" device=""/>
+<part name="JP2" library="pinhead" deviceset="PINHD-1X4" device=""/>
+<part name="GND4" library="supply1" deviceset="GND" device=""/>
+<part name="GND5" library="supply1" deviceset="GND" device=""/>
+<part name="JP3" library="pinhead" deviceset="PINHD-1X3" device=""/>
+<part name="GND6" library="supply1" deviceset="GND" device=""/>
 </parts>
 <sheets>
@@
 <instance part="JP1" gate="A" x="-68.58" y="50.8"/>
 <instance part="JP2" gate="A" x="-68.58" y="35.56"/>
+<instance part="GND4" gate="1" x="-83.82" y="53.34" rot="R270"/>
+<instance part="GND5" gate="1" x="-83.82" y="33.02" rot="R270"/>
+<instance part="JP3" gate="A" x="-68.58" y="73.66"/>
+<instance part="GND6" gate="1" x="-83.82" y="76.2" rot="R270"/>
 </instances>
 <busses>
@@
 <pinref part="GND3" gate="1" pin="GND"/>
 <wire x1="-15.24" y1="78.74" x2="-22.86" y2="78.74" width="0.1524" layer="91"/>
+</segment>
+<segment>
+<pinref part="JP1" gate="A" pin="2"/>
+<wire x1="-71.12" y1="53.34" x2="-78.74" y2="53.34" width="0.1524" layer="91"/>
+<wire x1="-78.74" y1="53.34" x2="-78.74" y2="50.8" width="0.1524" layer="91"/>
+<pinref part="JP1" gate="A" pin="3"/>
+<wire x1="-78.74" y1="50.8" x2="-71.12" y2="50.8" width="0.1524" layer="91"/>
+<pinref part="GND4" gate="1" pin="GND"/>
+<wire x1="-81.28" y1="53.34" x2="-78.74" y2="53.34" width="0.1524" layer="91"/>
+<junction x="-78.74" y="53.34"/>
+</segment>
+<segment>
+<pinref part="JP2" gate="A" pin="4"/>
+<pinref part="GND5" gate="1" pin="GND"/>
+<wire x1="-71.12" y1="33.02" x2="-81.28" y2="33.02" width="0.1524" layer="91"/>
+</segment>
+<segment>
+<pinref part="JP3" gate="A" pin="1"/>
+<pinref part="GND6" gate="1" pin="GND"/>
+<wire x1="-71.12" y1="76.2" x2="-81.28" y2="76.2" width="0.1524" layer="91"/>
 </segment>
 </net>
@@
 <segment>
 <pinref part="U1" gate="A" pin="1IN+"/>
-<wire x1="-15.24" y1="91.44" x2="-25.4" y2="91.44" width="0.1524" layer="91"/>
-<wire x1="-25.4" y1="91.44" x2="-25.4" y2="111.76" width="0.1524" layer="91"/>
-<wire x1="-25.4" y1="111.76" x2="73.66" y2="111.76" width="0.1524" layer="91"/>
-<pinref part="SV1" gate="G$1" pin="3"/>
-<wire x1="73.66" y1="86.36" x2="73.66" y2="111.76" width="0.1524" layer="91"/>
+<wire x1="-15.24" y1="91.44" x2="-30.48" y2="91.44" width="0.1524" layer="91"/>
+<wire x1="-30.48" y1="91.44" x2="-30.48" y2="22.86" width="0.1524" layer="91"/>
+<wire x1="-30.48" y1="22.86" x2="-91.44" y2="22.86" width="0.1524" layer="91"/>
+<wire x1="-91.44" y1="22.86" x2="-91.44" y2="35.56" width="0.1524" layer="91"/>
+<pinref part="JP2" gate="A" pin="3"/>
+<wire x1="-91.44" y1="35.56" x2="-71.12" y2="35.56" width="0.1524" layer="91"/>
+<pinref part="JP2" gate="A" pin="2"/>
+<wire x1="-71.12" y1="38.1" x2="-91.44" y2="38.1" width="0.1524" layer="91"/>
+<wire x1="-91.44" y1="38.1" x2="-91.44" y2="35.56" width="0.1524" layer="91"/>
+<junction x="-91.44" y="35.56"/>
 </segment>
 </net>
@@
 <pinref part="U1" gate="A" pin="VCC"/>
 <wire x1="-22.86" y1="99.06" x2="-15.24" y2="99.06" width="0.1524" layer="91"/>
+<wire x1="-22.86" y1="99.06" x2="-86.36" y2="99.06" width="0.1524" layer="91"/>
+<wire x1="-86.36" y1="99.06" x2="-86.36" y2="71.12" width="0.1524" layer="91"/>
+<pinref part="JP1" gate="A" pin="4"/>
+<wire x1="-86.36" y1="71.12" x2="-86.36" y2="48.26" width="0.1524" layer="91"/>
+<wire x1="-86.36" y1="48.26" x2="-71.12" y2="48.26" width="0.1524" layer="91"/>
+<pinref part="JP2" gate="A" pin="1"/>
+<wire x1="-71.12" y1="40.64" x2="-86.36" y2="40.64" width="0.1524" layer="91"/>
+<wire x1="-86.36" y1="40.64" x2="-86.36" y2="48.26" width="0.1524" layer="91"/>
+<junction x="-86.36" y="48.26"/>
+<junction x="-22.86" y="99.06"/>
+<pinref part="JP3" gate="A" pin="3"/>
+<wire x1="-71.12" y1="71.12" x2="-86.36" y2="71.12" width="0.1524" layer="91"/>
+<junction x="-86.36" y="71.12"/>
 </segment>
 </net>
+<net name="N$5" class="0">
+<segment>
+<pinref part="JP3" gate="A" pin="2"/>
+<wire x1="-71.12" y1="73.66" x2="-78.74" y2="73.66" width="0.1524" layer="91"/>
+<wire x1="-78.74" y1="73.66" x2="-78.74" y2="114.3" width="0.1524" layer="91"/>
+<pinref part="SV1" gate="G$1" pin="3"/>
+<wire x1="-78.74" y1="114.3" x2="73.66" y2="114.3" width="0.1524" layer="91"/>
+<wire x1="73.66" y1="114.3" x2="73.66" y2="86.36" width="0.1524" layer="91"/>
+</segment>
+</net>

Commit message: Some updates to the PCB, and a first list of required components.
Parts:
- added C2, C3: (no value), resistor:C-EUC0805
- added JP4: (no value), pinhead:PINHD-1X11
- added LED1, LED2: (no value), led:LEDCHIP-LED0805
- added R3, R4: (no value), resistor:R-EU_R0805
- C1: device resistor:CPOL-EU085CS-1AR -> resistor:CPOL-EU153CLV-0605
- IC1: value 74HC14D -> 74HC14N
- R1: device resistor:R-EU_R1005 -> resistor:R-EU_R0805
- R2: value 15k -> (none); device resistor:R-EU_R1005 -> resistor:R-EU_R0805
Connections:
- new net N$8: LED1.A, R3.1
- new net N$9: LED2.A, R4.1
- net GND: now also C2.2, C3.2, LED1.C, LED2.C
- net N$6: now also C2.1, R3.2
- net VCC: now also C3.1, R4.2

Commit message: replace input connector with a headerstrip so it can be clicked on a PI, and added a second strip that copies the input from the pie.
Parts:
- added SV2: (no value), pinhead:PINHD-2X13
- IC1: value 74HC14N -> 74HC14D
- SV1: device con-lstb:MA05-1 -> pinhead:PINHD-2X13
Connections:
- new net N$10: IC1E.O, SV1.12, SV2.12
- new net N$11: SV1.10, SV2.10
- new net N$12: SV1.16, SV2.16
- new net N$13: SV1.18, SV2.18
- new net N$14: SV1.22, SV2.22
- new net N$15: SV1.7, SV2.7
- new net N$16: SV1.24, SV2.24
- new net N$17: SV1.26, SV2.26
- new net N$18: SV1.3, SV2.3
- new net N$19: SV1.5, SV2.5
- new net N$21: SV1.13, SV2.13
- new net N$22: SV1.15, SV2.15
- new net N$23: SV1.19, SV2.19
- new net N$24: SV1.21, SV1.23, SV2.21, SV2.23
- net GND: now also SV1.14, SV1.20, SV1.25, SV1.6, SV1.9, SV2.14, SV2.20, SV2.25, SV2.6, SV2.9; no longer SV1.2
- net N$4: now also SV1.8, SV2.8; no longer IC1E.O, SV1.5
- net N$5: now also SV1.11, SV2.11; no longer SV1.3
- net N$6: now also SV1.2, SV2.2, SV2.4
- net VCC: now also SV1.17, SV2.1, SV2.17
Other:
- moved on the sheet: C3, LED2, R4

Commit message: Moved some stuff, tried adding a RJ1 connector as test.
Parts:
- added X1: 14867, con-4ucon:14867
Connections:
- net GND: now also X1.3
- net N$6: now also X1.4
Changed lines of the file:
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@@
 <part name="P+5" library="supply1" deviceset="VCC" device=""/>
 <part name="P+6" library="supply1" deviceset="VCC" device=""/>
+<part name="X1" library="con-4ucon" deviceset="14867" device=""/>
+<part name="GND20" library="supply1" deviceset="GND" device=""/>
 </parts>
 <sheets>
@@
 <instance part="P+5" gate="VCC" x="63.5" y="134.62" rot="R180"/>
 <instance part="P+6" gate="VCC" x="83.82" y="134.62" rot="R180"/>
+<instance part="X1" gate="G$1" x="157.48" y="139.7"/>
+<instance part="GND20" gate="1" x="149.86" y="139.7" rot="R270"/>
 </instances>
 <busses>
@@
 <pinref part="SV2" gate="A" pin="6"/>
 <wire x1="68.58" y1="154.94" x2="68.58" y2="149.86" width="0.1524" layer="91"/>
+</segment>
+<segment>
+<pinref part="X1" gate="G$1" pin="3"/>
+<pinref part="GND20" gate="1" pin="GND"/>
+<wire x1="152.4" y1="139.7" x2="154.94" y2="139.7" width="0.1524" layer="91"/>
 </segment>
 </net>
@@
 <wire x1="66.04" y1="149.86" x2="66.04" y2="160.02" width="0.1524" layer="91"/>
 <wire x1="66.04" y1="160.02" x2="63.5" y2="160.02" width="0.1524" layer="91"/>
-</segment>
-</net>
+<wire x1="0" y1="160.02" x2="0" y2="185.42" width="0.1524" layer="91"/>
+<wire x1="0" y1="185.42" x2="114.3" y2="185.42" width="0.1524" layer="91"/>
+<wire x1="114.3" y1="185.42" x2="114.3" y2="137.16" width="0.1524" layer="91"/>
+<pinref part="X1" gate="G$1" pin="4"/>
+<wire x1="114.3" y1="137.16" x2="154.94" y2="137.16" width="0.1524" layer="91"/>
+</segment>
+</net>

Commit message: Nieuwste revisie, connector omgedraaid zodat hij op de PI kan, RJ11 toegevoegd voor slimme meter.
Parts:
- removed SV2: (no value), pinhead:PINHD-2X13
Connections:
- removed net N$12: SV1.16, SV2.16
- removed net N$13: SV1.18, SV2.18
- removed net N$14: SV1.22, SV2.22
- removed net N$15: SV1.7, SV2.7
- removed net N$16: SV1.24, SV2.24
- removed net N$17: SV1.26, SV2.26
- removed net N$18: SV1.3, SV2.3
- removed net N$19: SV1.5, SV2.5
- removed net N$21: SV1.13, SV2.13
- removed net N$22: SV1.15, SV2.15
- removed net N$23: SV1.19, SV2.19
- removed net N$24: SV1.21, SV1.23, SV2.21, SV2.23
- net GND: no longer SV2.14, SV2.20, SV2.25, SV2.6, SV2.9
- net N$10: no longer SV2.12
- net N$11: now also IC1F.O; no longer SV2.10
- net N$4: now also IC1F.I, X1.1; no longer SV1.8, SV2.8
- net N$5: no longer SV2.11
- net N$6: no longer SV2.2, SV2.4
- net VCC: now also IC1A.I, IC1B.I, IC1C.I; no longer SV2.1, SV2.17
